Commit message: Update to code, increase simulation speed

File: AntModel/urdf/ant.urdf (robot description, URDF)
Before this commit: robot ant, 20 links, 19 joints
Links:
- link l_funiculus: geometry collision cylinder length=1.6 radius=0.05; visual cylinder length=1.6 radius=0.05
- link l_scape: geometry collision cylinder length=1.6 radius=0.05; visual cylinder length=1.6 radius=0.05
- link r_funiculus: geometry collision cylinder length=1.6 radius=0.05; visual cylinder length=1.6 radius=0.05
- link r_scape: geometry collision cylinder length=1.6 radius=0.05; visual cylinder length=1.6 radius=0.05
Joints:
- joint l_PS1: limit lower=-0.5 upper=1.2 effort=0.0 velocity=0.0 -> lower=-0.5 upper=0.77 effort=0.0 velocity=0.0
- joint l_PS2: limit lower=-1.2 upper=1.2 effort=0.0 velocity=0.0 -> lower=0.175 upper=1.7453 effort=0.0 velocity=0.0
- joint l_SF1: limit lower=-1.57 upper=1.374 effort=0.0 velocity=0.0 -> lower=-0.768 upper=1.047 effort=0.0 velocity=0.0; origin xyz=0.0 0.0 2 rpy=0.0 1.57 0 -> xyz=0.0 0.0 1.6 rpy=0.0 1.57 0
- joint l_end_joint: origin xyz=0.0 0.0 2.0 rpy=0.0 0.0 0.0 -> xyz=0.0 0.0 1.6 rpy=0.0 0.0 0.0
- joint r_PS1: limit lower=-0.5 upper=1.2 effort=0.0 velocity=0.0 -> lower=-0.5 upper=0.77 effort=0.0 velocity=0.0
- joint r_PS2: limit lower=-1.2 upper=1.2 effort=0.0 velocity=0.0 -> lower=0.175 upper=1.7453 effort=0.0 velocity=0.0
- joint r_SF1: limit lower=-1.57 upper=1.374 effort=0.0 velocity=0.0 -> lower=-0.768 upper=1.047 effort=0.0 velocity=0.0; origin xyz=0.0 0.0 2 rpy=0.0 1.57 0 -> xyz=0.0 0.0 1.6 rpy=0.0 1.57 0
- joint r_end_joint: origin xyz=0.0 0.0 2.0 rpy=0.0 0.0 0.0 -> xyz=0.0 0.0 1.6 rpy=0.0 0.0 0.0
